Commit message: laser enhanced

File: abrobot_description/urdf/robot2.xacro (robot description, xacro)
@@ -232,5 +232,5 @@
     </collision>
     <visual>
-      <origin xyz="-0.06 0 -0.05" rpy="0 0 0"/>
+      <origin xyz="0 0 -0.025" rpy="0 0 0"/>
       <geometry>
         <mesh filename="package://abrobot_description/meshes/rplidar.dae" scale="0.01 0.01 0.01" />
@@ -245,5 +245,5 @@
   <joint name="laser_joint" type="fixed">
     <axis xyz="0 1 0" />
-    <origin xyz=".15 0 .05" rpy="0 0 0"/>
+    <origin xyz=".15 0 .025" rpy="0 0 0"/>
     <parent link="base_link"/>
     <child link="base_laser"/>

Commit message: castor.dae and rplidar2.dae added wih different texture

File: abrobot_description/urdf/robot2.xacro (robot description, xacro)
@@ -66,5 +66,5 @@
         <origin xyz="0 0 0" rpy="-1.5707 0 1.5707" />
         <geometry>
-          <mesh filename="package://abrobot_description/meshes/28971-Caster-Wheel-Kit-v1.0.stl"/>
+          <mesh filename="package://abrobot_description/meshes/castor.dae"/>
         </geometry>
         <material name ="light_grey">
@@ -95,5 +95,5 @@
         <origin xyz="0 0 0" rpy="-1.5707 0 1.5707" />
         <geometry>
-          <mesh filename="package://abrobot_description/meshes/28971-Caster-Wheel-Kit-v1.0.stl"/>
+          <mesh filename="package://abrobot_description/meshes/castor.dae"/>
         </geometry>
         <material name ="light_grey">
@@ -234,5 +234,5 @@
       <origin xyz="0 0 -0.025" rpy="0 0 0"/>
       <geometry>
-        <mesh filename="package://abrobot_description/meshes/rplidar.dae" scale="0.01 0.01 0.01" />
+        <mesh filename="package://abrobot_description/meshes/rplidar2.dae" scale="0.01 0.01 0.01" />
       </geometry>
     </visual>

Commit message: xacro

File: abrobot_description/urdf/robot2.xacro (robot description, xacro)
@@ -184,5 +184,5 @@
         <origin xyz="0 0 0" rpy="0 1.5707 1.5707" />
         <geometry>
-          <cylinder radius="0.0782" length = "0.03175"/>
+          <cylinder radius="0.076" length = "0.03175"/>
         </geometry>
       </collision>
@@ -211,5 +211,5 @@
         <origin xyz="0 0 0" rpy="0 1.5707 1.5707" />
         <geometry>
-          <cylinder radius="0.0782" length = "0.03175"/>
+          <cylinder radius="0.076" length = "0.03175"/>
         </geometry>
       </collision>
@@ -232,7 +232,7 @@
     </collision>
     <visual>
-      <origin xyz="0 0 -0.025" rpy="0 0 0"/>
+      <origin xyz="0 0 -0.03" rpy="0 0 0"/>
       <geometry>
-        <mesh filename="package://abrobot_description/meshes/rplidar2.dae" scale="0.01 0.01 0.01" />
+        <mesh filename="package://abrobot_description/meshes/rplidar.stl" scale="0.01 0.01 0.01" />
       </geometry>
     </visual>

Commit message: changes for WebROS

File: abrobot_description/urdf/robot2.xacro (robot description, xacro)
@@ -17,5 +17,5 @@
           <cylinder length="0.0095" radius="0.2245"/>
         </geometry>
-        <material name ="veryDarkGrey" />
+        <material name ="White" />
       </visual>
       <collision>
